File: flex/flex.kicad_sch (KiCad schematic)
At the start: 27 parts, among them J1 Conn_01x06_Female, J2 Conn_01x03_Female, J3 Conn_01x01_Female, SW1 SW_Push, SW14 SW_Push, SW19 SW_Push, SW5 SW_Push, SW9 SW_Push

Commit message: licenses
Other:
- note added: "RGB"
- note added: "This work is licensed under a Creative Commons Attribution-NonCommercial-ShareAlike 4.0 International License."
- company: (none) -> bastard keyboards
- moved on the sheet: C1, C2, D1, D10, D11, D12, D13, D14, D19, D2, D3, D4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

Commit message: mousebites
Parts:
- added Mousebite1, Mousebite2, Mousebite3, Mousebite4: ~, customs:mousebite, symbol customs:mousebite

Commit message: update RGB
Parts:
- D10, D12, D2, D4, D7: footprint libs2:YS-SK6812MINI-E_REVERSE -> customs:SK6812_mini_e_corners
- D11, D13, D3, D6, D8: footprint libs2:YS-SK6812MINI-E_REVERSE_NO_EDGECUT -> customs:SK6812_mini_e_corners_noedgecuts
Changed lines of the file:
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@@
 			)
 		)
-		(property "Footprint" "libs2:YS-SK6812MINI-E_REVERSE"
+		(property "Footprint" "customs:SK6812_mini_e_corners"
 			(at 176.022 87.122 0)
 			(effects
@@
 			)
 		)
-		(property "Footprint" "libs2:YS-SK6812MINI-E_REVERSE"
+		(property "Footprint" "customs:SK6812_mini_e_corners"
 			(at 156.337 87.122 0)
 			(effects
@@
 			)
 		)
-		(property "Footprint" "libs2:YS-SK6812MINI-E_REVERSE"
+		(property "Footprint" "customs:SK6812_mini_e_corners"
 			(at 116.967 87.122 0)
 			(effects
@@
 			)
 		)
-		(property "Footprint" "libs2:YS-SK6812MINI-E_REVERSE_NO_EDGECUT"
+		(property "Footprint" "customs:SK6812_mini_e_corners_noedgecuts"
 			(at 116.967 109.982 0)
 			(effects
@@
 			)
 		)
-		(property "Footprint" "libs2:YS-SK6812MINI-E_REVERSE_NO_EDGECUT"
+		(property "Footprint" "customs:SK6812_mini_e_corners_noedgecuts"
 			(at 97.282 109.982 0)
 			(effects
@@
 			)
 		)
-		(property "Footprint" "libs2:YS-SK6812MINI-E_REVERSE_NO_EDGECUT"
+		(property "Footprint" "customs:SK6812_mini_e_corners_noedgecuts"
 			(at 136.652 109.982 0)
 			(effects
@@
 			)
 		)
-		(property "Footprint" "libs2:YS-SK6812MINI-E_REVERSE_NO_EDGECUT"
+		(property "Footprint" "customs:SK6812_mini_e_corners_noedgecuts"
 			(at 156.337 109.982 0)
 			(effects
@@
 			)
 		)
-		(property "Footprint" "libs2:YS-SK6812MINI-E_REVERSE"
+		(property "Footprint" "customs:SK6812_mini_e_corners"
 			(at 97.282 87.122 0)
 			(effects
@@
 			)
 		)
-		(property "Footprint" "libs2:YS-SK6812MINI-E_REVERSE_NO_EDGECUT"
+		(property "Footprint" "customs:SK6812_mini_e_corners_noedgecuts"
 			(at 176.022 109.982 0)
 			(effects
@@
 			)
 		)
-		(property "Footprint" "libs2:YS-SK6812MINI-E_REVERSE"
+		(property "Footprint" "customs:SK6812_mini_e_corners"
 			(at 136.652 87.122 0)
 			(effects
