File: flex/flex.kicad_pcb (KiCad board)
At the start: 2 copper layers, 74.1 x 41.5 mm, 29 parts, among them J1 Conn_01x06_Female, J2 Conn_01x03_Female, J3 Conn_01x01_Female, SW1 SW_Push, SW14 SW_Push, SW19 SW_Push, SW5 SW_Push, SW9 SW_Push

Commit message: mouse bites
Parts:
- added Mousebite1: ~, customs:mousebite, F.Cu at (65.8, 77.5)
- added Mousebite2: ~, customs:mousebite, F.Cu at (123.9, 79.9)
- added Mousebite3: ~, customs:mousebite, F.Cu at (67.3, 99.7)
- added Mousebite4: ~, customs:mousebite, F.Cu at (110.2, 93.0)
Other:
- outline, holes or cut-outs redrawn

Commit message: update RGB
Parts:
- added Mousebite2: ~, customs:mousebite, F.Cu at (2.20, 0.30)
- added Mousebite3: ~, customs:mousebite, F.Cu at (2.20, 1.90)
- added Mousebite4: ~, customs:mousebite, F.Cu at (2.20, 3.50)
- D10, D12, D2, D4, D7: footprint libs2:YS-SK6812MINI-E_REVERSE -> customs:SK6812_mini_e_corners
- D11, D13, D3, D6, D8: footprint libs2:YS-SK6812MINI-E_REVERSE_NO_EDGECUT -> customs:SK6812_mini_e_corners_noedgecuts

Commit message: silkscreen
Parts:
- moved Mousebite2 101.2 mm to (88.5, 53.1)
- moved Mousebite3 101.2 mm to (88.5, 54.7)
- moved Mousebite4 101.2 mm to (88.5, 56.3)
- moved D7 9.45 mm to (117.3, 73.0), turned to 165 degrees
- moved D8 9.45 mm to (117.3, 73.0), turned to 165 degrees
- moved D2 9.37 mm to (74.5, 93.7), turned to -170 degrees
- moved D3 9.37 mm to (74.5, 93.7), turned to -170 degrees
- moved D10 9.25 mm to (94.3, 69.9), turned to 180 degrees
- moved D11 9.25 mm to (94.3, 69.9), turned to 180 degrees
- moved D4 9.15 mm to (96.2, 91.8), turned to 180 degrees
- moved D6 9.15 mm to (96.2, 91.8), turned to 180 degrees
- moved D12 9.04 mm to (73.1, 71.9), turned to -170 degrees
- moved D13 9.04 mm to (73.1, 71.9), turned to -170 degrees
- moved SW5 0.17 mm to (73.9, 76.3), turned to -170 degrees
- moved SW14 0.14 mm to (115.9, 77.5), turned to 164 degrees
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Routing:
- net Gnd: track 139.2 -> 0.00 mm, vias 6 -> 0
- net Vcc: track 128.6 -> 0.00 mm, vias 6 -> 0
- net row1: track 121.7 -> 0.00 mm, vias 2 -> 0
- net col3: track 100.2 -> 0.00 mm, vias 3 -> 0
- net col6: track 98.0 -> 0.00 mm, vias 3 -> 0
- net Net-(D10-DOUT): track 52.0 -> 0.00 mm, vias 3 -> 0
- net Net-(D10-DIN): track 47.9 -> 0.00 mm, vias 2 -> 0
- net Net-(D4-DOUT): track 45.1 -> 0.00 mm, vias 3 -> 0
- net Net-(D12-DOUT): track 37.5 -> 0.00 mm, vias 1 -> 0
- net col4: track 32.5 -> 0.00 mm, vias 1 -> 0
- net Net-(D2-DOUT): track 26.5 -> 0.00 mm, vias 2 -> 0
- net Net-(D2-DIN): track 24.9 -> 0.00 mm, vias 2 -> 0
- net col5: track 21.5 -> 0.00 mm, vias 1 -> 0
- net Net-(D1-A): track 20.1 -> 0.00 mm, vias 1 -> 0
- net Net-(D14-A): track 18.0 -> 0.00 mm, vias 1 -> 0
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Other:
- board text added: "GITHUB.COM/BASTARDKB BASTARDKB.COM"
- board text added: "Licensed under CC BY-NC-SA 4.0 Copyright Q. Lebastard 2025"
- board text added: "REV 3.0"
- board text removed: "BASTARDKB.COM"
- board text removed: "C2R5"
- board text removed: "C3R5"
- board text removed: "C4R5"
- board text removed: "C5R5"
- board text removed: "C6R5"
- board text removed: "Do"
- board text removed: "GITHUB.COM/BASTARDKB"
- board text removed: "Licensed under CC BY-NC-SA 4.0 Copyright Quentin Lebastard 2022"
- board text removed: "REV 2.43"

Commit message: routing
Parts:
- removed the Mousebite2 at (88.5, 53.1)
- removed the Mousebite3 at (88.5, 54.7)
- removed the Mousebite4 at (88.5, 56.3)
Routing:
- net Vcc: track 0.00 -> 177.6 mm, vias 0 -> 5
- net Gnd: track 0.00 -> 155.9 mm, vias 0 -> 7
- net row1: track 0.00 -> 136.8 mm, vias 0 -> 5
- net Net-(D4-DOUT): track 0.00 -> 77.6 mm, vias 0 -> 4
- net col6: track 0.00 -> 75.1 mm, vias 0 -> 1
- net col3: track 0.00 -> 67.7 mm, vias 0 -> 1
- net Net-(D2-DOUT): track 0.00 -> 55.3 mm, vias 0 -> 4
- net col4: track 0.00 -> 32.3 mm, vias 0 -> 1
- net Net-(D12-DOUT): track 0.00 -> 28.3 mm, vias 0 -> 1
- net Net-(D10-DIN): track 0.00 -> 27.4 mm, vias 0 -> 3
- net Net-(D10-DOUT): track 0.00 -> 26.1 mm, vias 0 -> 3
- net col5: track 0.00 -> 21.4 mm, vias 0 -> 1
- net Net-(D9-A): track 0.00 -> 20.9 mm, vias 0 -> 1
- net Net-(D19-A): track 0.00 -> 20.5 mm, vias 0 -> 1
- net Net-(D5-A): track 0.00 -> 18.6 mm, vias 0 -> 1
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